File: intro_to_PCB.kicad_pcb (KiCad board)
At the start: 2 copper layers, 79 x 46.5 mm, 46 parts, among them J1 USB_C_Receptacle_USB2.0_16P, J2 Conn_01x16_Female, J3 Conn_01x16_Female, J4 ICSP, SW1 SW_Push, U1 ATmega328P-A, U2 LM1117DT-ADJ, U3 FT232RL, Y1 16MHz

Commit message: Add files via upload
Other:
- board size 79 x 46.5 mm -> 79.5 x 46.5 mm
Changed lines of the file:
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@@
 	(gr_poly
 		(pts
-			(xy 136 56.000768) (xy 136 92.000768) (xy 214.5 92.500768) (xy 215 46.500768) (xy 146 46.000768)
-			(xy 144.5 47.500768) (xy 144.5 54.500768) (xy 138 54.500768)
+			(xy 136 56.000768) (xy 135.5 92.5) (xy 214.5 92.500768) (xy 215 46.500768) (xy 146 46.000768) (xy 143.5 46)
+			(xy 139.5 46) (xy 136 46)
 		)
 		(stroke
@@
 		(polygon
 			(pts
-				(xy 135.5 45.5) (xy 135 93) (xy 214.5 92.5) (xy 215 46.5)
+				(xy 135.5 45.5) (xy 135 93) (xy 215 93) (xy 215 46.5)
 			)
 		)

Commit message: Add files via upload
Parts:
- moved C14 0.20 mm to (151.8, 51.8)
- moved C10 0.10 mm to (151.0, 82.2)
Other:
- board text added: "February 2025"
